File: Weekone/Weekone.kicad_sch (KiCad schematic)
At the start: 28 parts, among them IC1 AT42QT1011-MAHR, IC2 AT42QT1011-MAHR, IC3 AT42QT1011-MAHR, IC4 AT42QT1011-MAHR, IC5 AT42QT1011-MAHR, IC6 AT42QT1011-MAHR, IC7 AT42QT1011-MAHR, IC8 AT42QT1011-MAHR, IC9 AT42QT1011-MAHR, U1 XIAO-ESP32-C3-DIP

Commit message: wrapped up code and PCB design
Parts:
- C1, C2, C3, C4, C5, C6, C7, C8, C9: footprint 5pF cap:GRM022C81C222KE01L -> 5pf cap:GRM022C81C222KE01L
- C10, C11, C12, C13, C14, C15, C16, C17, C18: footprint 2nF cap:GCM21 -> 2nf cap:GCM21
- IC1, IC2, IC3, IC4, IC5, IC6, IC7, IC8, IC9: footprint Touch sensor IC:SON50P200X200X60-9N -> Weekone:SON50P200X200X60-9N
Connections:
- net GNDREF: now also C10.2, C11.2, C12.2, C13.2, C14.2, C15.2, C16.2, C17.2, C18.2, IC1.9 (EP), IC2.9 (EP), IC3.9 (EP), IC4.9 (EP), IC5.9 (EP), IC6.9 (EP), IC7.9 (EP), IC8.9 (EP), IC9.9 (EP)
- net at C1.1, IC1.1 (SNSK): now also C12.1
- net at IC2.1 (SNSK): now also C15.1, C2.1
- net at C7.1, IC7.1 (SNSK): now also C18.1
- net at C10.1: now also C3.1, IC3.1 (SNSK)
- net at C6.1, IC6.1 (SNSK): now also C11.1
- net at C9.1, IC9.1 (SNSK): now also C16.1
- net at IC5.1 (SNSK): now also C13.1, C5.1
- net at IC5.5 (OUT): now also U1.5 (GPIO6/D4/SDA)
- net at C8.1: now also C17.1, IC8.1 (SNSK)
- net at C4.1, IC4.1 (SNSK): now also C14.1
