File: Weekone/Weekone.kicad_pcb (KiCad board)
At the start: 2 copper layers, 80 x 50 mm, 28 parts, among them IC1 AT42QT1011-MAHR, IC2 AT42QT1011-MAHR, IC3 AT42QT1011-MAHR, IC4 AT42QT1011-MAHR, IC5 AT42QT1011-MAHR, IC6 AT42QT1011-MAHR, IC7 AT42QT1011-MAHR, IC8 AT42QT1011-MAHR, IC9 AT42QT1011-MAHR, U1 XIAO-ESP32-C3-DIP

Commit message: wrapped up code and PCB design
Parts:
- added .: LOGO, LOGO, F.Cu at (105.7, 141.6)
- C1, C2, C3, C4, C5, C6, C7, C8, C9: footprint 5pF cap:GRM022C81C222KE01L -> 5pf cap:GRM022C81C222KE01L
- C10, C11, C12, C13, C14, C15, C16, C17, C18: footprint 2nF cap:GCM21 -> 2nf cap:GCM21
- IC1, IC2, IC3, IC4, IC5, IC6, IC7, IC8, IC9: footprint Touch sensor IC:SON50P200X200X60-9N -> Weekone:SON50P200X200X60-9N
- moved C16 58.8 mm to (165.1, 132.4), turned to 180 degrees
- moved C10 57.8 mm to (131.3, 132.4), turned to 180 degrees
- moved C11 57.2 mm to (148.2, 136.2), turned to 90 degrees
- moved IC9 47.2 mm to (169.9, 137.8)
- moved C3 44.1 mm to (136.2, 135.9)
- moved IC6 43.2 mm to (154.9, 137.8)
- moved C17 43.1 mm to (163.4, 120.9), turned to 180 degrees
- moved C9 42.3 mm to (169.9, 135.4)
- moved IC3 42.2 mm to (136.2, 138.3)
- moved C13 42.1 mm to (153.9, 116.4), turned to 180 degrees
- moved C6 40.9 mm to (154.9, 135.4)
- moved IC8 36.9 mm to (169.8, 121.8)
- moved C15 33.8 mm to (133.4, 115.6), turned to 180 degrees
- moved C2 32.5 mm to (136.4, 119.9)
- moved IC5 31.8 mm to (155.0, 121.8)
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Connections:
- C10 pad 1: unconnected-(C10-Pad1) -> Net-(IC3-SNSK)
- C10 pad 2: unconnected-(C10-Pad2) -> GNDREF
- C11 pad 1: unconnected-(C11-Pad1) -> Net-(IC6-SNSK)
- C11 pad 2: unconnected-(C11-Pad2) -> GNDREF
- C12 pad 1: unconnected-(C12-Pad1) -> Net-(IC1-SNSK)
- C12 pad 2: unconnected-(C12-Pad2) -> GNDREF
- C13 pad 1: unconnected-(C13-Pad1) -> Net-(IC5-SNSK)
- C13 pad 2: unconnected-(C13-Pad2) -> GNDREF
- C14 pad 1: unconnected-(C14-Pad1) -> Net-(IC4-SNSK)
- C14 pad 2: unconnected-(C14-Pad2) -> GNDREF
- C15 pad 1: unconnected-(C15-Pad1) -> Net-(IC2-SNSK)
- C15 pad 2: unconnected-(C15-Pad2) -> GNDREF
- C16 pad 1: unconnected-(C16-Pad1) -> Net-(IC9-SNSK)
- C16 pad 2: unconnected-(C16-Pad2) -> GNDREF
- C17 pad 1: unconnected-(C17-Pad1) -> Net-(IC8-SNSK)
- C17 pad 2: unconnected-(C17-Pad2) -> GNDREF
- C18 pad 1: unconnected-(C18-Pad1) -> Net-(IC7-SNSK)
- C18 pad 2: unconnected-(C18-Pad2) -> GNDREF
- C2 pad 1: unconnected-(C2-Pad1) -> Net-(IC2-SNSK)
- C5 pad 1: unconnected-(C5-Pad1) -> Net-(IC5-SNSK)
- C8 pad 1: unconnected-(C8-Pad1) -> Net-(IC8-SNSK)
- IC1 pad 9: unconnected-(IC1-EP-Pad9) -> GNDREF
- IC2 pad 1: unconnected-(IC2-SNSK-Pad1) -> Net-(IC2-SNSK)
- IC2 pad 9: unconnected-(IC2-EP-Pad9) -> GNDREF
- IC3 pad 9: unconnected-(IC3-EP-Pad9) -> GNDREF
- IC4 pad 9: unconnected-(IC4-EP-Pad9) -> GNDREF
- IC5 pad 1: unconnected-(IC5-SNSK-Pad1) -> Net-(IC5-SNSK)
- IC5 pad 5: unconnected-(IC5-OUT-Pad5) -> Net-(IC5-OUT)
- IC5 pad 9: unconnected-(IC5-EP-Pad9) -> GNDREF
- IC6 pad 9: unconnected-(IC6-EP-Pad9) -> GNDREF
- IC7 pad 9: unconnected-(IC7-EP-Pad9) -> GNDREF
- IC8 pad 1: unconnected-(IC8-SNSK-Pad1) -> Net-(IC8-SNSK)
- IC8 pad 9: unconnected-(IC8-EP-Pad9) -> GNDREF
- IC9 pad 9: unconnected-(IC9-EP-Pad9) -> GNDREF
- U1 pad 5: unconnected-(U1-GPIO6/D4/SDA-Pad5) -> Net-(IC5-OUT)
Routing:
- net GNDREF: track 0.00 -> 238.9 mm, vias 0 -> 8
- net +3.3V: track 0.00 -> 193.5 mm, vias 0 -> 6
- net Net-(IC5-OUT): track 0.00 -> 90.4 mm
- net Net-(IC6-OUT): track 0.00 -> 74.3 mm
- net Net-(IC4-OUT): track 0.00 -> 70.6 mm, vias 0 -> 2
- net Net-(IC7-OUT): track 0.00 -> 66.2 mm, vias 0 -> 2
- net Net-(IC9-OUT): track 0.00 -> 62.2 mm, vias 0 -> 1
- net Net-(IC8-OUT): track 0.00 -> 58.1 mm, vias 0 -> 1
- net Net-(IC3-OUT): track 0.00 -> 57.0 mm
- net Net-(IC1-OUT): track 0.00 -> 53.6 mm, vias 0 -> 2
- net Net-(IC2-OUT): track 0.00 -> 44.4 mm, vias 0 -> 2
- net Net-(IC3-SNSK): track 0.00 -> 15.4 mm, vias 0 -> 2
- net Net-(IC1-SNSK): track 0.00 -> 12.9 mm, vias 0 -> 2
- net Net-(IC2-SNSK): track 0.00 -> 11.2 mm, vias 0 -> 2
- net Net-(IC7-SNSK): track 0.00 -> 10.9 mm, vias 0 -> 2
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
Commit message: Note in README
Routing:
- net Net-(IC7-SNSK): track 10.9 -> 11.6 mm
Changed lines of the file:
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@@
 			(outputformat 1)
 			(mirror no)
-			(drillshape 1)
+			(drillshape 0)
 			(scaleselection 1)
-			(outputdirectory "")
+			(outputdirectory "./")
 		)
 	)
@@
 			(at 0 0 0)
 			(layer "F.SilkS")
+			(hide yes)
 			(effects
 				(font
@@
 	)
 	(segment
-		(start 165.45 104.2)
-		(end 164.6 104.2)
+		(start 168.475 107.225)
+		(end 165.45 104.2)
 		(width 0.2)
 		(layer "B.Cu")
@@
 	)
 	(segment
-		(start 169.2 107.95)
-		(end 165.45 104.2)
+		(start 168.475 105.5)
+		(end 168.475 107.225)
+		(width 0.2)
+		(layer "B.Cu")
+		(net 34)
+	)
+	(segment
+		(start 165.45 104.2)
+		(end 164.6 104.2)
 		(width 0.2)
 		(layer "B.Cu")
